Commit message: Ajout de rtabmap_slam dans le Launch

File: src/mentorpi_simulation/urdf/mecanum.xacro (robot description, xacro)
@@ -167,4 +167,11 @@
     <axis xyz="0 0 0"/>
   </joint>
+  <link name="depth_cam_optical_frame"/>
+  <joint name="depth_cam_optical_joint" type="fixed">
+    <parent link="depth_cam"/>
+    <child link="depth_cam_optical_frame"/>
+    <!-- rotation standard optique: roll=-pi/2, pitch=0, yaw=-pi/2 -->
+    <origin xyz="0 0 0" rpy="-1.5707963267948966 0 -1.5707963267948966"/>
+  </joint>
   <link name="lidar_frame">
     <inertial>

File: src/mentorpi_simulation/urdf/ros2_control.xacro (robot description, xacro)
@@ -121,4 +121,32 @@
                 </sensor>
             </gazebo>
+            <gazebo reference="depth_cam">
+                <sensor name="depth_camera" type="rgbd_camera">
+                    <always_on>true</always_on>
+                    <update_rate>30.0</update_rate>
+                    <visualize>true</visualize>
+                    <!-- Topic racine côté Gazebo -->
+                    <topic>/depth_cam</topic>
+                    <camera>
+                        <horizontal_fov>1.047</horizontal_fov>
+                        <image>
+                            <width>640</width>
+                            <height>480</height>
+                            <format>R8G8B8</format>
+                        </image>
+                        <clip>
+                            <near>0.05</near>
+                            <far>10.0</far>
+                        </clip>
+                        <depth_camera>
+                            <clip>
+                                <near>0.05</near>
+                                <far>10.0</far>
+                            </clip>
+                        </depth_camera>
+                        <optical_frame_id>depth_cam_optical_frame</optical_frame_id>
+                    </camera>
+                </sensor>
+            </gazebo>
         </xacro:if>
         <xacro:if value="${use_sim}">
